File: hardware/BMP180 breakout v02.brd (EAGLE design)
At the start: 15.2 x 15.2 mm, 15 parts, among them U1 BMP180

Commit message: minor changes to eagle files re. group review
Parts:
- R1, R2: value (none) -> 4.7K
Changed lines of the file:
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@@
 <layer number="14" name="Route14" color="1" fill="6" visible="no" active="no"/>
 <layer number="15" name="Route15" color="4" fill="6" visible="no" active="no"/>
-<layer number="16" name="Bottom" color="1" fill="1" visible="yes" active="yes"/>
+<layer number="16" name="Bottom" color="1" fill="1" visible="no" active="yes"/>
 <layer number="17" name="Pads" color="2" fill="1" visible="yes" active="yes"/>
 <layer number="18" name="Vias" color="2" fill="1" visible="yes" active="yes"/>
@@
 <layer number="27" name="tValues" color="7" fill="1" visible="no" active="yes"/>
 <layer number="28" name="bValues" color="7" fill="1" visible="no" active="yes"/>
-<layer number="29" name="tStop" color="7" fill="3" visible="yes" active="yes"/>
+<layer number="29" name="tStop" color="7" fill="3" visible="no" active="yes"/>
 <layer number="30" name="bStop" color="7" fill="6" visible="no" active="yes"/>
 <layer number="31" name="tCream" color="7" fill="4" visible="yes" active="yes"/>
@@
 <layer number="49" name="Reference" color="7" fill="1" visible="no" active="yes"/>
 <layer number="50" name="dxf" color="7" fill="1" visible="no" active="no"/>
-<layer number="51" name="tDocu" color="6" fill="1" visible="yes" active="yes"/>
+<layer number="51" name="tDocu" color="6" fill="1" visible="no" active="yes"/>
 <layer number="52" name="bDocu" color="7" fill="1" visible="no" active="yes"/>
 <layer number="53" name="tGND_GNDA" color="7" fill="9" visible="no" active="no"/>
@@
 <element name="U1" library="mike-temp" package="BMP180" value="BMP180" x="7.62" y="7.62"/>
 <element name="SJ1" library="mike-temp" package="SJ_3_PASTE1&amp;2&amp;3" value="" x="12.7" y="8.255"/>
-<element name="R1" library="SparkFun-Passives" package="0603-RES" value="" x="13.97" y="5.08" rot="R90"/>
-<element name="R2" library="SparkFun-Passives" package="0603-RES" value="" x="11.43" y="5.08" rot="R90"/>
+<element name="R1" library="SparkFun-Passives" package="0603-RES" value="4.7K" x="13.97" y="5.08" rot="R90"/>
+<element name="R2" library="SparkFun-Passives" package="0603-RES" value="4.7K" x="11.43" y="5.08" rot="R90"/>
 <element name="C1" library="SparkFun-Capacitors" package="0603-CAP" value="0.1uF" x="7.62" y="11.1125"/>
 <element name="C2" library="SparkFun-Capacitors" package="0603-CAP" value="0.1uF" x="3.81" y="5.08" rot="R270"/>
@@
 <contactref element="C1" pad="2"/>
 <contactref element="C2" pad="2"/>
-<polygon width="0.2032" layer="16">
+<polygon width="0.2032" layer="16" isolate="0.3048">
 <vertex x="0" y="15.24"/>
 <vertex x="0" y="0"/>
@@
 <vertex x="15.24" y="15.24"/>
 </polygon>
-<polygon width="0.2032" layer="1">
+<polygon width="0.2032" layer="1" isolate="0.3048">
 <vertex x="0" y="15.24"/>
 <vertex x="0" y="0"/>

Commit message: final proto hardware, initial library
Library copied and renamed from BMP085 floating-point library (see USB
Weather Board)
Connections:
- removed net VCC: C1.1, C3.A, JP1.2, SJ1.2, SJ2.1, U1.2
- removed net VCCIO: C2.1, JP1.1, SJ2.2, U1.3
- new net VDD: C1.1, C3.A, JP1.2, SJ2.1, U1.2
- new net VDDIO: C2.1, JP1.1, SJ1.2, SJ2.2, U1.3
Routing:
- net VCC: track 27.2 -> 0.00 mm, vias 1 -> 0
- net VDDIO: track 0.00 -> 23.3 mm, vias 0 -> 2
- net VDD: track 0.00 -> 20.9 mm, vias 0 -> 1
- net VCCIO: track 10.6 -> 0.00 mm
Changed lines of the file:
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@@
 <setting verticaltext="up"/>
 </settings>
-<grid distance="0.05" unitdist="inch" unit="inch" style="lines" multiple="2" display="yes" altdistance="0.005" altunitdist="inch" altunit="inch"/>
+<grid distance="0.05" unitdist="inch" unit="inch" style="lines" multiple="2" display="yes" altdistance="0.0125" altunitdist="inch" altunit="inch"/>
 <layers>
 <layer number="1" name="Top" color="4" fill="1" visible="yes" active="yes"/>
@@
 <layer number="14" name="Route14" color="1" fill="6" visible="no" active="no"/>
 <layer number="15" name="Route15" color="4" fill="6" visible="no" active="no"/>
-<layer number="16" name="Bottom" color="1" fill="1" visible="no" active="yes"/>
+<layer number="16" name="Bottom" color="1" fill="1" visible="yes" active="yes"/>
 <layer number="17" name="Pads" color="2" fill="1" visible="yes" active="yes"/>
 <layer number="18" name="Vias" color="2" fill="1" visible="yes" active="yes"/>
-<layer number="19" name="Unrouted" color="6" fill="1" visible="yes" active="yes"/>
+<layer number="19" name="Unrouted" color="6" fill="1" visible="no" active="yes"/>
 <layer number="20" name="Dimension" color="15" fill="1" visible="yes" active="yes"/>
 <layer number="21" name="tPlace" color="16" fill="1" visible="yes" active="yes"/>
@@
 <layer number="29" name="tStop" color="7" fill="3" visible="no" active="yes"/>
 <layer number="30" name="bStop" color="7" fill="6" visible="no" active="yes"/>
-<layer number="31" name="tCream" color="7" fill="4" visible="yes" active="yes"/>
+<layer number="31" name="tCream" color="7" fill="4" visible="no" active="yes"/>
 <layer number="32" name="bCream" color="7" fill="5" visible="no" active="yes"/>
 <layer number="33" name="tFinish" color="6" fill="3" visible="no" active="yes"/>
@@
 <layer number="106" name="bPlate" color="7" fill="1" visible="no" active="yes"/>
 <layer number="107" name="Crop" color="7" fill="1" visible="no" active="yes"/>
+<layer number="116" name="Patch_BOT" color="9" fill="4" visible="no" active="yes"/>
 <layer number="121" name="_tsilk" color="7" fill="1" visible="no" active="yes"/>
 <layer number="122" name="_bsilk" color="7" fill="1" visible="no" active="yes"/>
@@
 <layer number="220" name="220bmp" color="21" fill="1" visible="no" active="no"/>
 <layer number="221" name="221bmp" color="22" fill="1" visible="no" active="no"/>
+<layer number="222" name="222bmp" color="23" fill="1" visible="no" active="no"/>
 <layer number="223" name="223bmp" color="24" fill="1" visible="no" active="no"/>
 <layer number="224" name="224bmp" color="25" fill="1" visible="no" active="no"/>
@@
 <wire x1="15.24" y1="15.24" x2="0" y2="15.24" width="0.2032" layer="20"/>
 <wire x1="0" y1="15.24" x2="0" y2="0" width="0.2032" layer="20"/>
-<text x="4.2545" y="13.0175" size="1.27" layer="21" font="vector" ratio="15">BMP180</text>
+<text x="4.2545" y="13.6525" size="1.27" layer="21" font="vector" ratio="15">BMP180</text>
 <text x="4.60375" y="2.2225" size="1.27" layer="21" font="vector" ratio="15">+</text>
 <text x="1.905" y="2.38125" size="1.016" layer="21" font="vector" ratio="15">IO</text>
@@
 <wire x1="7.62" y1="3.81" x2="10.16" y2="1.27" width="0.3048" layer="1"/>
 </signal>
-<signal name="VCC">
+<signal name="VDD">
 <contactref element="SJ2" pad="1"/>
-<contactref element="SJ1" pad="2"/>
 <contactref element="U1" pad="2"/>
 <contactref element="C3" pad="A"/>
@@
 <wire x1="6.77" y1="11.1125" x2="6.77" y2="9.8425" width="0.3048" layer="1"/>
 <wire x1="6.77" y1="9.8425" x2="7.62" y2="9.8425" width="0.3048" layer="1"/>
-<wire x1="7.62" y1="9.8425" x2="12.065" y2="9.8425" width="0.3048" layer="1"/>
-<wire x1="12.065" y1="9.8425" x2="12.7" y2="9.2075" width="0.3048" layer="1"/>
-<wire x1="12.7" y1="9.2075" x2="12.7" y2="8.255" width="0.3048" layer="1"/>
 <wire x1="0.8581" y1="5.08" x2="0.8581" y2="6.09685" width="0.3048" layer="1"/>
 <wire x1="0.8581" y1="6.09685" x2="1.42875" y2="6.6675" width="0.3048" layer="1"/>
@@
 <wire x1="2.3525" y1="6.6675" x2="3.94" y2="8.255" width="0.3048" layer="1"/>
 <wire x1="7.62" y1="9.07" x2="7.62" y2="9.8425" width="0.3048" layer="1"/>
-<contactref element="JP1" pad="2"/>
-<wire x1="5.08" y1="1.27" x2="2.54" y2="3.81" width="0.3048" layer="16"/>
 <wire x1="2.54" y1="3.81" x2="2.54" y2="8.255" width="0.3048" layer="16"/>
 <via x="2.54" y="8.255" extent="1-16" drill="0.508"/>
 <wire x1="2.54" y1="8.255" x2="3.94" y2="8.255" width="0.3048" layer="1"/>
+<contactref element="JP1" pad="2"/>
+<wire x1="2.54" y1="3.81" x2="5.08" y2="1.27" width="0.3048" layer="16"/>
 </signal>
 <signal name="GND">
@@
 <vertex x="15.24" y="15.24"/>
 </polygon>
-<via x="10.16" y="7.62" extent="1-16" drill="0.508"/>
-<via x="10.16" y="11.1125" extent="1-16" drill="0.508"/>
-<via x="1.27" y="10.16" extent="1-16" drill="0.508"/>
-</signal>
-<signal name="VCCIO">
+<via x="10.4775" y="7.62" extent="1-16" drill="0.508"/>
+<via x="8.5725" y="12.7" extent="1-16" drill="0.508"/>
+<via x="0.9525" y="9.8425" extent="1-16" drill="0.508"/>
+</signal>
+<signal name="VDDIO">
 <contactref element="SJ2" pad="2"/>
 <contactref element="U1" pad="3"/>
 <contactref element="C2" pad="1"/>
-<wire x1="3.81" y1="5.93" x2="6.12" y2="8.24" width="0.3048" layer="1"/>
-<wire x1="6.12" y1="8.24" x2="6.12" y2="9.07" width="0.3048" layer="1"/>
 <contactref element="JP1" pad="1"/>
 <wire x1="2.54" y1="1.27" x2="2.54" y2="5.08" width="0.3048" layer="1"/>
 <wire x1="2.54" y1="5.08" x2="1.6819" y2="5.08" width="0.3048" layer="1"/>
 <wire x1="3.81" y1="5.93" x2="3.009" y2="5.93" width="0.3048" layer="1"/>
-<wire x1="3.009" y1="5.93" x2="2.667" y2="5.588" width="0.3048" layer="1"/>
+<wire x1="3.009" y1="5.93" x2="2.54" y2="5.461" width="0.3048" layer="1"/>
 <wire x1="2.54" y1="5.08" x2="2.54" y2="5.461" width="0.3048" layer="1"/>
-<wire x1="2.54" y1="5.461" x2="2.667" y2="5.588" width="0.3048" layer="1"/>
+<contactref element="SJ1" pad="2"/>
+<wire x1="6.12" y1="9.07" x2="5.08" y2="8.03" width="0.3048" layer="1"/>
+<wire x1="5.08" y1="8.03" x2="5.08" y2="6.35" width="0.3048" layer="1"/>
+<wire x1="5.08" y1="5.93" x2="5.08" y2="5.08" width="0.3048" layer="1"/>
+<wire x1="5.08" y1="5.08" x2="5.3975" y2="4.7625" width="0.3048" layer="1"/>
+<via x="5.3975" y="4.7625" extent="1-16" drill="0.508"/>
+<wire x1="3.81" y1="5.93" x2="5.08" y2="5.93" width="0.3048" layer="1"/>
+<wire x1="5.08" y1="5.93" x2="5.08" y2="6.35" width="0.3048" layer="1"/>
+<wire x1="5.3975" y1="4.7625" x2="10.4775" y2="9.8425" width="0.3048" layer="16"/>
+<via x="10.4775" y="9.8425" extent="1-16" drill="0.508"/>
+<wire x1="10.4775" y1="9.8425" x2="12.065" y2="9.8425" width="0.3048" layer="1"/>
+<wire x1="12.065" y1="9.8425" x2="12.7" y2="9.2075" width="0.3048" layer="1"/>
+<wire x1="12.7" y1="9.2075" x2="12.7" y2="8.255" width="0.3048" layer="1"/>
 </signal>
 </signals>
