File: hardware/BMP180 breakout v02.sch (EAGLE design)
At the start: 15 parts, among them U1 BMP180

Commit message: minor changes to eagle files re. group review
Parts:
- R1, R2: value (none) -> 4.7K
Changed lines of the file:
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@@
 <part name="U1" library="mike-temp" deviceset="BMP180" device=""/>
 <part name="SJ1" library="mike-temp" deviceset="SOLDERJUMPER_2WAY" device="PASTE1&amp;2&amp;3"/>
-<part name="R1" library="SparkFun-Passives" deviceset="RESISTOR" device="0603-RES"/>
-<part name="R2" library="SparkFun-Passives" deviceset="RESISTOR" device="0603-RES"/>
+<part name="R1" library="SparkFun-Passives" deviceset="RESISTOR" device="0603-RES" value="4.7K"/>
+<part name="R2" library="SparkFun-Passives" deviceset="RESISTOR" device="0603-RES" value="4.7K"/>
 <part name="C1" library="SparkFun-Capacitors" deviceset="CAP" device="0603-CAP" value="0.1uF"/>
 <part name="C2" library="SparkFun-Capacitors" deviceset="CAP" device="0603-CAP" value="0.1uF"/>
@@
 <part name="JP1" library="mike-temp" deviceset="M05" device="_ROUNDONLY_NOSILK"/>
 <part name="SJ2" library="mike-temp" deviceset="SOLDERJUMPER" device="NC" value=""/>
-<part name="SUPPLY1" library="SparkFun-Aesthetics" deviceset="VCC" device=""/>
 <part name="SUPPLY2" library="SparkFun-Aesthetics" deviceset="VCC" device=""/>
 <part name="SUPPLY3" library="SparkFun-Aesthetics" deviceset="VCC" device="" value="VCCIO"/>
@@
 <instance part="JP1" gate="G$1" x="40.64" y="96.52"/>
 <instance part="SJ2" gate="1" x="160.02" y="116.84"/>
-<instance part="SUPPLY1" gate="1" x="144.78" y="127"/>
 <instance part="SUPPLY2" gate="1" x="154.94" y="127"/>
 <instance part="SUPPLY3" gate="1" x="165.1" y="127"/>
@@
 <wire x1="91.44" y1="104.14" x2="91.44" y2="101.6" width="0.1524" layer="91"/>
 <junction x="91.44" y="101.6"/>
-<label x="81.28" y="101.6" size="1.778" layer="95" rot="R180" xref="yes"/>
+<label x="81.28" y="101.6" size="1.27" layer="95" rot="R180" xref="yes"/>
 </segment>
 <segment>
@@
 <wire x1="101.6" y1="104.14" x2="101.6" y2="96.52" width="0.1524" layer="91"/>
 <junction x="101.6" y="96.52"/>
-<label x="81.28" y="96.52" size="1.778" layer="95" rot="R180" xref="yes"/>
+<label x="81.28" y="96.52" size="1.27" layer="95" rot="R180" xref="yes"/>
 </segment>
 <segment>
@@
 <segment>
 <pinref part="SJ2" gate="1" pin="1"/>
-<wire x1="154.94" y1="114.3" x2="154.94" y2="116.84" width="0.1524" layer="91"/>
 <wire x1="154.94" y1="116.84" x2="154.94" y2="127" width="0.1524" layer="91"/>
 <junction x="154.94" y="116.84"/>
@@
 <pinref part="C3" gate="G$1" pin="+"/>
 <pinref part="C1" gate="G$1" pin="1"/>
-<pinref part="SUPPLY1" gate="1" pin="VCC"/>
-<wire x1="144.78" y1="127" x2="144.78" y2="101.6" width="0.1524" layer="91"/>
-<wire x1="154.94" y1="114.3" x2="154.94" y2="101.6" width="0.1524" layer="91"/>
+<wire x1="154.94" y1="116.84" x2="154.94" y2="101.6" width="0.1524" layer="91"/>
 <junction x="154.94" y="101.6"/>
 </segment>

Commit message: final proto hardware, initial library
Library copied and renamed from BMP085 floating-point library (see USB
Weather Board)
Connections:
- removed net VCC: C1.1, C3.+, JP1.2, SJ1.2, SJ2.1, U1.VDD
- removed net VCCIO: C2.1, JP1.1, SJ2.2, U1.VDDIO
- new net VDD: C1.1, C3.+, JP1.2, SJ2.1, U1.VDD
- new net VDDIO: C2.1, JP1.1, SJ1.2, SJ2.2, U1.VDDIO
Other:
- note added: "AND VDDIO TOGETHER"
- note added: "ON I2C LINES"
- note added: "SHORT BOTH SIDES OF SJ1"
- note added: "SHORT SJ2 TO CONNECT VDD"
- note added: "TO ENABLE PULL-UP RESISTORS"
Changed lines of the file:
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@@
 <part name="JP1" library="mike-temp" deviceset="M05" device="_ROUNDONLY_NOSILK"/>
 <part name="SJ2" library="mike-temp" deviceset="SOLDERJUMPER" device="NC" value=""/>
-<part name="SUPPLY2" library="SparkFun-Aesthetics" deviceset="VCC" device=""/>
-<part name="SUPPLY3" library="SparkFun-Aesthetics" deviceset="VCC" device="" value="VCCIO"/>
+<part name="SUPPLY2" library="SparkFun-Aesthetics" deviceset="VCC" device="" value="VDD"/>
+<part name="SUPPLY3" library="SparkFun-Aesthetics" deviceset="VCC" device="" value="VDDIO"/>
 <part name="GND1" library="SparkFun-Aesthetics" deviceset="GND" device=""/>
 <part name="GND2" library="SparkFun-Aesthetics" deviceset="GND" device=""/>
 <part name="GND3" library="SparkFun-Aesthetics" deviceset="GND" device=""/>
 <part name="GND4" library="SparkFun-Aesthetics" deviceset="GND" device=""/>
-<part name="SUPPLY4" library="SparkFun-Aesthetics" deviceset="VCC" device=""/>
+<part name="SUPPLY4" library="SparkFun-Aesthetics" deviceset="VCC" device="" value="VDDIO"/>
 <part name="LOGO1" library="SparkFun-Aesthetics" deviceset="LOGO-SFE" device="NW2"/>
 <part name="LOGO2" library="SparkFun-Aesthetics" deviceset="OSHW-LOGO" device="S"/>
@@
 <rectangle x1="159.385" y1="116.205" x2="160.655" y2="117.475" layer="94"/>
 <text x="172.72" y="7.62" size="2.54" layer="94">M Grusin</text>
+<text x="104.14" y="119.38" size="1.778" layer="97">SHORT BOTH SIDES OF SJ1</text>
+<text x="104.14" y="116.84" size="1.778" layer="97">TO ENABLE PULL-UP RESISTORS</text>
+<text x="104.14" y="114.3" size="1.778" layer="97">ON I2C LINES</text>
+<text x="167.64" y="119.38" size="1.778" layer="97">SHORT SJ2 TO CONNECT VDD</text>
+<text x="167.64" y="116.84" size="1.778" layer="97">AND VDDIO TOGETHER</text>
 </plain>
 <instances>
@@
 </segment>
 </net>
-<net name="VCC" class="0">
+<net name="VDD" class="0">
 <segment>
 <pinref part="SJ2" gate="1" pin="1"/>
@@
 <wire x1="154.94" y1="116.84" x2="154.94" y2="101.6" width="0.1524" layer="91"/>
 <junction x="154.94" y="101.6"/>
-</segment>
-<segment>
-<pinref part="SJ1" gate="G$1" pin="2"/>
-<pinref part="SUPPLY4" gate="1" pin="VCC"/>
-<wire x1="96.52" y1="127" x2="96.52" y2="124.46" width="0.1524" layer="91"/>
 </segment>
 <segment>
@@
 </segment>
 </net>
-<net name="VCCIO" class="0">
+<net name="VDDIO" class="0">
 <segment>
 <pinref part="SJ2" gate="1" pin="2"/>
@@
 <label x="50.8" y="91.44" size="1.27" layer="95" xref="yes"/>
 </segment>
+<segment>
+<pinref part="SJ1" gate="G$1" pin="2"/>
+<pinref part="SUPPLY4" gate="1" pin="VCC"/>
+<wire x1="96.52" y1="127" x2="96.52" y2="124.46" width="0.1524" layer="91"/>
+</segment>
 </net>
